Commit message: fine for gmapping and amcl

File: amr_description/urdf/amr_simply.urdf (robot description, URDF)
Before this commit: robot amr, 4 links, 3 joints
Joints:
- joint hokuyo_joint: axis (none) -> 0 0 1; origin xyz=0.35 -0.28 0.09 rpy=0.0 0.0 -0.785 -> xyz=0.355 -0.275 0.09 rpy=0.0 0.0 -0.7854
- joint lw_joint: axis 0 1 0 -> 0 0 1; origin xyz=0 0.225 0.1 rpy=0 0 0 -> xyz=0 0.225 0.1 rpy=-1.5707963267949 0 0
- joint rw_joint: axis 0 1 0 -> 0 0 -1; origin xyz=0 -0.225 0.1 rpy=0 0 0 -> xyz=0 -0.225 0.1 rpy=1.5707963267949 0 0
